Commit message: Added zed camera urdf, and updated camera calibration to use it.

File: src/site_configs/atomos_xlink_hw_config/description/motiv_xlink_atomos.mock.urdf (robot description, URDF)
Before this commit: robot xlink, 23 links, 22 joints
Links:
- added link calibration_tool_frame
- added link calibration_tool_link; visual mesh filename=file://$(find atomos_xlink_hw_config)/description/assets/ca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
- added link estimated_zed_base_frame
- added link zed_camera_center; collision mesh filename=file:///opt/ros/humble/share/zed_msgs/meshes/zed2i.stl; visual mesh filename=file:///opt/ros/humble/share/zed_msgs/meshes/zed2i.stl
- added link zed_camera_link
- added link zed_left_camera_frame
- added link zed_left_camera_optical_frame
- added link zed_right_camera_frame
- added link zed_right_camera_optical_frame
Joints:
- added joint calibration_tool_frame_joint: type fixed, parent calibration_tool_link, child calibration_tool_frame, origin xyz=0 -0.09325 -0.01 rpy=0 ${pi} ${pi}
- added joint calibration_tool_joint: type fixed, parent grasp_link, child calibration_tool_link, origin xyz=0 0 0.011 rpy=0 0 0
- added joint estimated_zed_base_frame_joint: type fixed, parent base_link, child estimated_zed_base_frame, origin xyz=0.3 -0.2 -0.05 rpy=1.542 -1.542 0
- added joint parent_zed_camera_link_joint: type fixed, parent estimated_zed_base_frame, child zed_camera_link, origin xyz=0 0 0 rpy=0 0 0
- added joint zed_camera_center_joint: type fixed, parent zed_camera_link, child zed_camera_center, origin xyz=0 0 0.015 rpy=0 0.0 0
- added joint zed_left_camera_joint: type fixed, parent zed_camera_center, child zed_left_camera_frame, origin xyz=-0.01 0.06 0 rpy=0 0 0
- added joint zed_left_camera_optical_joint: type fixed, parent zed_left_camera_frame, child zed_left_camera_optical_frame, origin xyz=0 0 0 rpy=-1.5707963267948966 0.0 -1.5707963267948966
- added joint zed_right_camera_joint: type fixed, parent zed_camera_center, child zed_right_camera_frame, origin xyz=-0.01 -0.06 0 rpy=0 0 0
- added joint zed_right_camera_optical_joint: type fixed, parent zed_right_camera_frame, child zed_right_camera_optical_frame, origin xyz=0 0 0 rpy=-1.5707963267948966 0.0 -1.5707963267948966

Commit message: Fix teleoperate and URDF meshes in motiv_xlink_atomos.mock

File: src/site_configs/atomos_xlink_hw_config/description/motiv_xlink_atomos.mock.urdf (robot description, URDF)
Before this commit: robot xlink, 32 links, 31 joints
Links:
- link base_link: geometry collision mesh filename=package://xlink_description/meshes/collision/base_link.stl; visual mesh filename=package://xlink_description/meshes/visual/base_link.dae
- link left_finger_link: geometry collision mesh filename=package://xlink_gripper_description/meshes/collision/basic_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; visual mesh filename=package://xlink_gripper_description/meshes/visual/basic_fin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
- link left_inner_link: geometry collision mesh filename=package://xlink_gripper_description/meshes/collision/inner_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; visual mesh filename=package://xlink_gripper_description/meshes/visual/inner_lin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
- link left_outer_link: geometry collision mesh filename=package://xlink_gripper_description/meshes/collision/outer_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; visual mesh filename=package://xlink_gripper_description/meshes/visual/outer_lin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
- link link_1: geometry collision mesh filename=package://xlink_description/meshes/collision/link_1.stl; visual mesh filename=package://xlink_description/meshes/visual/link_1.dae
- link link_2: geometry collision mesh filename=package://xlink_description/meshes/collision/link_2.stl; visual mesh filename=package://xlink_description/meshes/visual/link_2.dae
- link link_3: geometry collision mesh filename=package://xlink_description/meshes/collision/link_3.stl; visual mesh filename=package://xlink_description/meshes/visual/link_3.dae
- link link_4: geometry collision mesh filename=package://xlink_description/meshes/collision/link_4.stl; visual mesh filename=package://xlink_description/meshes/visual/link_4.dae
- link link_5: geometry collision mesh filename=package://xlink_description/meshes/collision/link_5.stl; visual mesh filename=package://xlink_description/meshes/visual/link_5.dae
- link link_6: geometry collision mesh filename=package://xlink_description/meshes/collision/link_6.stl; visual mesh filename=package://xlink_description/meshes/visual/link_6.dae
- link link_7: geometry collision mesh filename=package://xlink_description/meshes/collision/link_7.stl; visual mesh filename=package://xlink_description/meshes/visual/link_7.dae
- link right_finger_link: geometry collision mesh filename=package://xlink_gripper_description/meshes/collision/basic_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; visual mesh filename=package://xlink_gripper_description/meshes/visual/basic_fin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
- link right_inner_link: geometry collision mesh filename=package://xlink_gripper_description/meshes/collision/inner_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; visual mesh filename=package://xlink_gripper_description/meshes/visual/inner_lin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
- link right_outer_link: geometry collision mesh filename=package://xlink_gripper_description/meshes/collision/outer_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; visual mesh filename=package://xlink_gripper_description/meshes/visual/outer_lin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
- link servicer_sled_link: geometry collision mesh filename=file://$(find atomos_xlink_hw_config)/description/assets/cr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 scale=0.1 0.1 0.1; visual mesh filename=file://$(find atomos_xlink_hw_config)/description/assets/cr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 scale=0.1 0.1 0.1
- link xlink_gripper_base: geometry collision mesh filename=package://xlink_gripper_description/meshes/collision/grippe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; visual mesh filename=package://xlink_gripper_description/meshes/visual/gripper_b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

Commit message: xlink works, adding waypoints and test objectives.

File: src/site_configs/atomos_xlink_hw_config/description/motiv_xlink_atomos.mock.urdf (robot description, URDF)
Before this commit: robot xlink, 32 links, 31 joints
Links:
- added link back; collision box size=0.2 2.0 2.0; visual box size=0.2 2.0 2.0
- added link floor; collision box size=4.0 4.0 0.2; visual box size=4.0 4.0 0.2
- added link tank_air_hoses; collision box size=0.15 0.15 0.15; visual box size=0.15 0.15 0.15
Joints:
- added joint back_joint: type fixed, parent servicer_sled_link, child back, origin xyz=-0.11 0 0 rpy=0 0 0
- added joint floor_joint: type fixed, parent servicer_sled_link, child floor, origin xyz=0 0 -0.57 rpy=0 0 0
- added joint tank_air_hoses_joint: type fixed, parent servicer_sled_link, child tank_air_hoses, origin xyz=0.26 -0.38 -0.33 rpy=0 0 0
- joint base_joint: origin xyz=0 0 0 rpy=-1.5707963267948966 0.0 -1.5707963267948966 -> xyz=0 0 0 rpy=-3.14159 -1.5707963267948966 0.0
- joint estimated_zed_base_frame_joint: origin xyz=0.3 -0.2 -0.05 rpy=1.542 -1.542 0 -> xyz=-0.035 -0.39 0.24 rpy=0 0 0; parent base_link -> servicer_sled_link

Commit message: Day 1.

File: src/site_configs/atomos_xlink_hw_config/description/motiv_xlink_atomos.mock.urdf (robot description, URDF)
Before this commit: robot xlink, 35 links, 34 joints
Joints:
- joint estimated_zed_base_frame_joint: origin xyz=-0.035 -0.39 0.24 rpy=0 0 0 -> xyz=-0.050 -0.39 0.24 rpy=0 0 0

Commit message: Update urdf
Add rafti fingers, comment out calibration tool and camera.

File: src/site_configs/atomos_xlink_hw_config/description/motiv_xlink_atomos.mock.urdf (robot description, URDF)
Before this commit: robot xlink, 35 links, 34 joints
Links:
- removed link calibration_tool_frame
- removed link calibration_tool_link
- removed link wrist_mounted_camera_bottom_screw_frame
- removed link wrist_mounted_camera_link
- added link left_rafti_finger_link; collision mesh filename=package://atomos_xlink_hw_config/description/assets/xlink_r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; visual mesh filename=package://atomos_xlink_hw_config/description/assets/xlink_r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
- added link right_rafti_finger_link; collision mesh filename=package://atomos_xlink_hw_config/description/assets/xlink_r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; visual mesh filename=package://atomos_xlink_hw_config/description/assets/xlink_r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
Joints:
- removed joint calibration_tool_frame_joint
- removed joint calibration_tool_joint
- removed joint wrist_mounted_camera_joint
- removed joint wrist_mounted_camera_link_joint
- added joint left_rafti_finger_joint: type fixed, parent left_finger_link, child left_rafti_finger_link, origin xyz=0 0 0 rpy=3.14259 0 0
- added joint right_rafti_finger_joint: type fixed, parent right_finger_link, child right_rafti_finger_link, origin xyz=0 0 0 rpy=3.14259 0 0

Commit message: Update zed camera location

File: src/site_configs/atomos_xlink_hw_config/description/motiv_xlink_atomos.mock.urdf (robot description, URDF)
Before this commit: robot xlink, 33 links, 32 joints
Joints:
- joint estimated_zed_base_frame_joint: origin xyz=-0.050 -0.39 0.24 rpy=0 0 0 -> xyz=-0.024939 -0.37902 0.21445 rpy=0 0 0

Commit message: swap rafti fingers for calibration tool.

File: src/site_configs/atomos_xlink_hw_config/description/motiv_xlink_atomos.mock.urdf (robot description, URDF)
Before this commit: robot xlink, 33 links, 32 joints
Links:
- removed link left_rafti_finger_link
- removed link right_rafti_finger_link
- added link calibration_tool_frame
- added link calibration_tool_link; visual mesh filename=file://$(find atomos_xlink_hw_config)/description/assets/ca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
Joints:
- removed joint left_rafti_finger_joint
- removed joint right_rafti_finger_joint
- added joint calibration_tool_frame_joint: type fixed, parent calibration_tool_link, child calibration_tool_frame, origin xyz=0 -0.09325 -0.01 rpy=0 ${pi} ${pi}
- added joint calibration_tool_joint: type fixed, parent grasp_link, child calibration_tool_link, origin xyz=0 0 0.011 rpy=0 0 0

Commit message: hw changes

File: src/site_configs/atomos_xlink_hw_config/description/motiv_xlink_atomos.mock.urdf (robot description, URDF)
Before this commit: robot xlink, 33 links, 32 joints
Links:
- link calibration_tool_link: geometry collision mesh filename=file://$(find atomos_xlink_hw_config)/description/assets/ca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; visual mesh filename=file://$(find atomos_xlink_hw_config)/description/assets/ca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

Commit message: Update urdf with driver updates

File: src/site_configs/atomos_xlink_hw_config/description/motiv_xlink_atomos.mock.urdf (robot description, URDF)
Before this commit: robot xlink, 33 links, 32 joints
Links:
- removed link calibration_tool_frame
- added link end_effector_attach_link
- added link xlink_gripper_edge
- link base_link: mass 0.7823 -> 0.7557; geometry collision mesh filename=file:///home/dwyackzan/moveit_pro_source/install/xlink_desc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; visual mesh filename=file:///home/dwyackzan/moveit_pro_source/install/xlink_desc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
- link left_finger_link: geometry collision mesh filename=file:///home/dwyackzan/moveit_pro_source/install/xlink_grip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; visual mesh filename=file:///home/dwyackzan/moveit_pro_source/install/xlink_grip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
- link left_inner_link: geometry collision mesh filename=file:///home/dwyackzan/moveit_pro_source/install/xlink_grip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; visual mesh filename=file:///home/dwyackzan/moveit_pro_source/install/xlink_grip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
- link left_outer_link: geometry collision mesh filename=file:///home/dwyackzan/moveit_pro_source/install/xlink_grip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; visual mesh filename=file:///home/dwyackzan/moveit_pro_source/install/xlink_grip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
- link link_1: mass 5.5103 -> 4.9525; geometry collision mesh filename=file:///home/dwyackzan/moveit_pro_source/install/xlink_desc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; visual mesh filename=file:///home/dwyackzan/moveit_pro_source/install/xlink_desc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
- link link_2: geometry collision mesh filename=file:///home/dwyackzan/moveit_pro_source/install/xlink_desc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; visual mesh filename=file:///home/dwyackzan/moveit_pro_source/install/xlink_desc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
- link link_3: mass 5.3096 -> 4.7009; geometry collision mesh filename=file:///home/dwyackzan/moveit_pro_source/install/xlink_desc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; visual mesh filename=file:///home/dwyackzan/moveit_pro_source/install/xlink_desc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
- link link_4: mass .5653 -> .5703; geometry collision mesh filename=file:///home/dwyackzan/moveit_pro_source/install/xlink_desc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; visual mesh filename=file:///home/dwyackzan/moveit_pro_source/install/xlink_desc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
- link link_5: mass 5.3096 -> 4.7009; geometry collision mesh filename=file:///home/dwyackzan/moveit_pro_source/install/xlink_desc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; visual mesh filename=file:///home/dwyackzan/moveit_pro_source/install/xlink_desc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
- link link_6: mass .5653 -> .5703; geometry collision mesh filename=file:///home/dwyackzan/moveit_pro_source/install/xlink_desc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; visual mesh filename=file:///home/dwyackzan/moveit_pro_source/install/xlink_desc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
- link link_7: mass 3.6704 -> 3.2507; geometry collision mesh filename=file:///home/dwyackzan/moveit_pro_source/install/xlink_desc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; visual mesh filename=file:///home/dwyackzan/moveit_pro_source/install/xlink_desc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
- link right_finger_link: geometry collision mesh filename=file:///home/dwyackzan/moveit_pro_source/install/xlink_grip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; visual mesh filename=file:///home/dwyackzan/moveit_pro_source/install/xlink_grip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
- link right_inner_link: geometry collision mesh filename=file:///home/dwyackzan/moveit_pro_source/install/xlink_grip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; visual mesh filename=file:///home/dwyackzan/moveit_pro_source/install/xlink_grip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
- link right_outer_link: geometry collision mesh filename=file:///home/dwyackzan/moveit_pro_source/install/xlink_grip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; visual mesh filename=file:///home/dwyackzan/moveit_pro_source/install/xlink_grip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
- link xlink_gripper_base: geometry collision mesh filename=file:///home/dwyackzan/moveit_pro_source/install/xlink_grip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; visual mesh filename=file:///home/dwyackzan/moveit_pro_source/install/xlink_grip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
Joints:
- removed joint calibration_tool_frame_joint
- added joint end_effector_attach_joint: type fixed, parent fts_link, child end_effector_attach_link, origin xyz=0 0 -0.02857 rpy=3.1416 0 3.1416
- added joint xlink_gripper_edge_joint: type fixed, parent xlink_gripper_base, child xlink_gripper_edge, origin xyz=0 0 0.14935 rpy=0 0 0
- joint base_joint: parent servicer_sled_link -> world
- joint fts_joint: origin xyz=0 0 0.26643 rpy=3.1416 0 1.5708 -> xyz=0 0 0.26643 rpy=3.1416 0 3.1416
- joint gripper_base_joint: origin xyz=0 0 -0.029 rpy=0 3.141592653589793 0 -> xyz=0 0 0 rpy=0 0 0; parent fts_link -> end_effector_attach_link
- joint gripper_joint: limit lower=0 upper=1.0 effort=500.0 velocity=1.0 -> lower=0 upper=0.82 effort=500.0 velocity=1.0
- joint joint_1: origin xyz=0 0 0.111 rpy=0 0 0 -> xyz=0 0 0.387 rpy=0 0 0
- joint joint_2: origin xyz=0 0 0.276 rpy=3.1416 -1.5708 3.1416 -> xyz=0 -.159 0 rpy=1.5708 0 0
- joint joint_3: origin xyz=0 0 0.159 rpy=0 1.5708 0 -> xyz=0 .328 0 rpy=-1.5708 0 0
- joint joint_4: origin xyz=0 0 0.32809 rpy=0 -1.5708 3.1416 -> xyz=0 .155 0 rpy=-1.5708 0 0
- joint joint_5: origin xyz=0 0 0.155 rpy=0 -1.5708 3.1416 -> xyz=0 -.325 0 rpy=1.5708 0 0
- joint joint_6: origin xyz=0 0 0.325 rpy=2.93874 -1.5708 -2.93874 -> xyz=0 -.155 0 rpy=1.5708 0 0
- joint joint_7: origin xyz=0 0 0.155 rpy=0 1.5708 0 -> xyz=0 0 0 rpy=-1.5708 0 0
- joint left_finger_joint: limit lower=0 upper=1.0 effort=500.0 velocity=1.0 -> lower=0 upper=0.82 effort=500.0 velocity=1.0
- joint left_inner_joint: limit lower=0 upper=1.0 effort=500.0 velocity=1.0 -> lower=0 upper=0.82 effort=500.0 velocity=1.0
- joint right_finger_joint: limit lower=0 upper=1.0 effort=500.0 velocity=1.0 -> lower=0 upper=0.82 effort=500.0 velocity=1.0
- joint right_inner_joint: limit lower=0 upper=1.0 effort=500.0 velocity=1.0 -> lower=0 upper=0.82 effort=500.0 velocity=1.0
- joint right_outer_joint: limit lower=0 upper=1.0 effort=500.0 velocity=1.0 -> lower=0 upper=0.82 effort=500.0 velocity=1.0

Commit message: Fix absolute paths in urdf

File: src/site_configs/atomos_xlink_hw_config/description/motiv_xlink_atomos.mock.urdf (robot description, URDF)
Before this commit: robot xlink, 34 links, 33 joints
Links:
- link base_link: geometry collision mesh filename=package://xlink_description/meshes/collision/base_link.stl; visual mesh filename=package://xlink_description/meshes/visual/base_link.dae
- link left_finger_link: geometry collision mesh filename=package://xlink_gripper_description/meshes/collision/basic_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; visual mesh filename=package://xlink_gripper_description/meshes/visual/basic_fin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
- link left_inner_link: geometry collision mesh filename=package://xlink_gripper_description/meshes/collision/inner_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; visual mesh filename=package://xlink_gripper_description/meshes/visual/inner_lin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
- link left_outer_link: geometry collision mesh filename=package://xlink_gripper_description/meshes/collision/outer_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; visual mesh filename=package://xlink_gripper_description/meshes/visual/outer_lin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
- link link_1: geometry collision mesh filename=package://xlink_description/meshes/collision/link_1.stl; visual mesh filename=package://xlink_description/meshes/visual/link_1.dae
- link link_2: geometry collision mesh filename=package://xlink_description/meshes/collision/link_2.stl; visual mesh filename=package://xlink_description/meshes/visual/link_2.dae
- link link_3: geometry collision mesh filename=package://xlink_description/meshes/collision/link_3.stl; visual mesh filename=package://xlink_description/meshes/visual/link_3.dae
- link link_4: geometry collision mesh filename=package://xlink_description/meshes/collision/link_4.stl; visual mesh filename=package://xlink_description/meshes/visual/link_4.dae
- link link_5: geometry collision mesh filename=package://xlink_description/meshes/collision/link_5.stl; visual mesh filename=package://xlink_description/meshes/visual/link_5.dae
- link link_6: geometry collision mesh filename=package://xlink_description/meshes/collision/link_6.stl; visual mesh filename=package://xlink_description/meshes/visual/link_6.dae
- link link_7: geometry collision mesh filename=package://xlink_description/meshes/collision/link_7.stl; visual mesh filename=package://xlink_description/meshes/visual/link_7.dae
- link right_finger_link: geometry collision mesh filename=package://xlink_gripper_description/meshes/collision/basic_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; visual mesh filename=package://xlink_gripper_description/meshes/visual/basic_fin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
- link right_inner_link: geometry collision mesh filename=package://xlink_gripper_description/meshes/collision/inner_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; visual mesh filename=package://xlink_gripper_description/meshes/visual/inner_lin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
- link right_outer_link: geometry collision mesh filename=package://xlink_gripper_description/meshes/collision/outer_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; visual mesh filename=package://xlink_gripper_description/meshes/visual/outer_lin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
- link xlink_gripper_base: geometry collision mesh filename=package://xlink_gripper_description/meshes/collision/grippe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; visual mesh filename=package://xlink_gripper_description/meshes/visual/gripper_b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

Commit message: Fix zed mesh paths in urdf

File: src/site_configs/atomos_xlink_hw_config/description/motiv_xlink_atomos.mock.urdf (robot description, URDF)
Before this commit: robot xlink, 34 links, 33 joints
Links:
- link zed_camera_center: geometry collision mesh filename=package://zed_msgs/meshes/zed2i.stl; visual mesh filename=package://zed_msgs/meshes/zed2i.stl

Commit message: Launch & description file updates

File: src/site_configs/atomos_xlink_hw_config/description/motiv_xlink_atomos.mock.urdf (robot description, URDF)
Before this commit: robot xlink, 34 links, 33 joints
Links:
- removed link calibration_tool_link
- added link left_rafti_finger_link; collision mesh filename=package://atomos_xlink_hw_config/description/assets/xlink_r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; visual mesh filename=package://atomos_xlink_hw_config/description/assets/xlink_r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
- added link right_rafti_finger_link; collision mesh filename=package://atomos_xlink_hw_config/description/assets/xlink_r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; visual mesh filename=package://atomos_xlink_hw_config/description/assets/xlink_r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
Joints:
- removed joint calibration_tool_joint
- added joint left_rafti_finger_joint: type fixed, parent left_finger_link, child left_rafti_finger_link, origin xyz=0 0 0 rpy=3.14259 0 0
- added joint right_rafti_finger_joint: type fixed, parent right_finger_link, child right_rafti_finger_link, origin xyz=0 0 0 rpy=3.14259 0 0
- joint base_joint: origin xyz=0 0 0 rpy=-3.14159 -1.5707963267948966 0.0 -> xyz=0 0 0 rpy=1.5708 0.0 1.5708
- joint estimated_zed_base_frame_joint: origin xyz=-0.024939 -0.37902 0.21445 rpy=0 0 0 -> xyz=-0.024658 -0.37036 0.21471 rpy=0 0 0

Commit message: Update urdf to rotated mount and add track only objective

File: src/site_configs/atomos_xlink_hw_config/description/motiv_xlink_atomos.mock.urdf (robot description, URDF)
Before this commit: robot xlink, 35 links, 34 joints
Joints:
- joint base_joint: origin xyz=0 0 0 rpy=1.5708 0.0 1.5708 -> xyz=0 0 0 rpy=3.14159265 -1.57079633 0

Commit message: Tested and validated values with new camera position.

File: src/site_configs/atomos_xlink_hw_config/description/motiv_xlink_atomos.mock.urdf (robot description, URDF)
Before this commit: robot xlink, 35 links, 34 joints
Joints:
- joint estimated_zed_base_frame_joint: origin xyz=-0.024658 -0.37036 0.21471 rpy=0 0 0 -> xyz=-0.024752 -0.378874 0.481702 rpy=0 0 0
- joint floor_joint: origin xyz=0 0 -0.57 rpy=0 0 0 -> xyz=0 0 -0.47 rpy=0 0 0
